Commit message: 尝试修复ik问题，重新写了mjcf文件，但是发现其不能正常通过mujocoinclude引用

File: DISCOVERSE/models/urdf/xbot_arm.bak.urdf (robot description, URDF)
Before this commit: robot xarm, 10 links, 9 joints
Joints:
- joint arm_2_joint: limit lower=-2.094 upper=1.5707963267948966 effort=100 velocity=0.35 -> lower=-2.094 upper=1.57079632679 effort=100 velocity=0.35
